File: ndsbreakoutboard/ndsbreakoutboard.kicad_pcb (KiCad board)
At the start: 2 copper layers, 27.3 x 30.5 mm, 19 parts, among them J14 Conn_01x01_Female, U1 ndsPADS

Commit message: rough push
Parts:
- moved 3.3V 58.8 mm to (111.0, 21.7)
- moved J14 56.9 mm to (88.8, 21.7)
- moved CS2 47.9 mm to (93.4, 21.7)
- moved CS1 47.9 mm to (90.3, 21.7)
- moved D0 47.9 mm to (97.5, 21.7)
- moved D2 47.9 mm to (100.6, 21.7)
- moved D6 47.8 mm to (106.6, 21.7)
- moved D4 47.8 mm to (103.6, 21.7)
- moved D7 47.8 mm to (108.1, 21.7)
- moved GND 47.6 mm to (85.6, 21.7)
- moved RES 41.3 mm to (91.8, 21.7)
- moved IRQ 41.3 mm to (94.9, 21.7)
- moved CLK 41.3 mm to (87.3, 21.7)
- moved D5 41.2 mm to (105.1, 21.7)
- moved D3 41.2 mm to (102.1, 21.7)
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Routing:
- net Net-(J15-Pad1): track 9.77 -> 80.4 mm, vias 0 -> 1
- net Net-(J14-Pad1): track 9.43 -> 66.4 mm
- net Net-(J6-Pad1): track 18.5 -> 66.4 mm
- net Net-(J4-Pad1): track 18.5 -> 66.4 mm
- net Net-(J8-Pad1): track 18.6 -> 66.5 mm
- net Net-(J13-Pad1): track 18.6 -> 66.5 mm
- net Net-(J10-Pad1): track 18.7 -> 66.5 mm
- net Net-(J12-Pad1): track 18.9 -> 66.5 mm
- net Net-(J2-Pad1): track 20.7 -> 66.4 mm
- net Net-(J7-Pad1): track 25.2 -> 66.7 mm
- net Net-(J5-Pad1): track 25.1 -> 66.5 mm
- net Net-(J3-Pad1): track 25.1 -> 66.4 mm
- net Net-(J9-Pad1): track 25.2 -> 66.5 mm
- net Net-(J1-Pad1): track 25.1 -> 66.4 mm
- net Net-(J11-Pad1): track 25.3 -> 66.5 mm
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- removed copper zone on B.Cu, net Net-(GNDLine1-Pad1)
Other:
- board size 27.3 x 30.5 mm -> 27.3 x 72.1 mm
- net class Default removed
- board text added: "Nintendo DS & 3DS Breakout Board github.com/pedro-javierf/dscartpcb modded by haifisch :)"
- board text removed: "Nintendo DS & 3DS Breakout Board github.com/pedro-javierf/dscartpcb"
